File: design/drv8301.sch (KiCad schematic (older format))
At the start: 25 parts

Commit message: 2020-12-21
Parts:
- added C? (x2): 2.2uF, Capacitor_SMD:C_0603_1608Metric, symbol Device:C
- added C?: 100uF, Capacitor_Tantalum_SMD:CP_EIA-6032-20_AVX-F, symbol Device:CP
- added C?: 100nF, Capacitor_SMD:C_0603_1608Metric, symbol Device:C
- added Q?: DMN62D0UW-7, Package_TO_SOT_SMD:SOT-323_SC-70, symbol Transistor_FET:DMN62D0UW-7
- added R? (x2): 2k2, Resistor_SMD:R_0603_1608Metric, symbol Device:R
- added R? (x2): 39k, Resistor_SMD:R_0603_1608Metric, symbol Device:R
- added U?: TC2117-3.3VDBTR, Package_TO_SOT_SMD:SOT-223-3_TabPin2, symbol TC211733VDBTR:TC2117-3.3VDBTR
- added U?: M74VHC1GT66DTT1G, AnalogSwitch:M74VHC1GT66DTT1G, symbol M74VHC1GT66DTT1G:M74VHC1GT66DTT1G
- D?: value D -> TVS 5V
Connections:
- net +3V3: now also C?.1, C?.1, U?.2 (VOUT), U?.5 (VCC)
- net +5V: now also C?.1, Q?.1 (G), U?.3 (VIN)
- net GND: now also U?.57 (EPAD), C?.2, C?.2, C?.2, R?.1, R?.2, U?.1 (GND), U?.2 (OUT/INYA), U?.3 (GND)
- net SH_A: now also R?.1
- net SUPPLY: now also R?.1
- new net: Q?.3 (D), R?.2
- new net: C?.2, U?.1 (IN/OUTXA)
- new net SENS_A: C?.1, R?.2, R?.2
- new net SENS_FILTERED: U?.4 (ON/OFF)
- new net SENS_SUPPLY: Q?.2 (S), R?.1

Commit message: 210104
Parts:
- added C38, C39: 100nF, Capacitor_SMD:C_0603_1608Metric, symbol Device:C
- added R25, R27: 39k, Resistor_SMD:R_0603_1608Metric, symbol Device:R
- added R26, R28: 2k2, Resistor_SMD:R_0603_1608Metric, symbol Device:R
- added U10, U11: M74VHC1GT66DTT1G, AnalogSwitch:M74VHC1GT66DTT1G, symbol M74VHC1GT66DTT1G:M74VHC1GT66DTT1G
- R23: renamed from R?; MPN CPF0603B39KE1 -> ERJ-3EKF3902V
- U7: renamed from U?; footprint DCA56_6P35X3P61 -> Package_SO:HTSSOP-56-1EP_6.1x14mm_P0.5mm_EP3.61x6.35mm
- gave numbers to parts that had none: 34
Connections:
- net +3V3: now also U10.5 (VCC), U11.5 (VCC)
- net GND: now also R26.1, R28.1, U10.2 (OUT/INYA), U10.3 (GND), U11.2 (OUT/INYA), U11.3 (GND)
- net SENS_FILTERED: now also U10.4 (ON/OFF), U11.4 (ON/OFF)
- net SH_B: now also R25.1
- net SH_C: now also R27.1
- new net: C38.2, U10.1 (IN/OUTXA)
- new net: C39.2, U11.1 (IN/OUTXA)
- new net SENS_B: C38.1, R25.2, R26.2
- new net SENS_C: C39.1, R27.2, R28.2
Other:
- moved on the sheet: C37, R23, R24, U9
