File: design/power.sch (KiCad schematic (older format))
At the start: 2 parts

Commit message: power board design 1
Parts:
- added C1, C2, C3, C4, C5, C6: 4.7uF_100V, Capacitor_SMD:C_1210_3225Metric, symbol Device:C
- added C10, C11, C12: 1nF, Capacitor_SMD:C_0603_1608Metric, symbol Device:C
- added C13, C14, C15: 15nF, Capacitor_SMD:C_0603_1608Metric, symbol Device:C
- added C16, C17: 680uF_63V, Capacitor_SMD:CP_Elec_18x22, symbol Device:CP1
- added C18, C7, C8, C9: 2.2uF, Capacitor_SMD:C_0603_1608Metric, symbol Device:C
- added P1: SUPPLY, PADS:HighCurrent_WithHoles_400mils, symbol PADS:POWER
- added P2: PH_A, symbol PADS:POWER
- added P3: PH_B, symbol PADS:POWER
- added P4: PH_C, symbol PADS:POWER
- added P5: GND, PADS:HighCurrent_WithHoles_400mils, symbol PADS:POWER
- added Q1, Q2, Q4, Q5: IRF7749L2TRPBF, IRF7749L2TRPBF:Infineon-IRF7749L2TRPBF-0-0-0, symbol IRF7749L2TRPBF:IRF7749L2TRPBF
- added R1, R2, R3, R7, R8, R9: 4.7R, Resistor_SMD:R_0603_1608Metric, symbol Device:R
- added R10, R11, R12: 1k, Resistor_SMD:R_0603_1608Metric, symbol Device:R
- added R13: NTC 10k, Resistor_SMD:R_0603_1608Metric, symbol Device:R
- added R14: 10k, Resistor_SMD:R_0603_1608Metric, symbol Device:R
- added R4, R5, R6: 0.0005R, HighCurrentShunt:RESC3216X105N, symbol HCS1206FTL500:HCS1206FTL500
- added U1, U2, U3: AD8418, Package_SO:MSOP-8_3x3mm_P0.65mm, symbol Amplifier_Current:AD8418
- added U4, U5, U6: M74VHC1GT66DTT1G, AnalogSwitch:M74VHC1GT66DTT1G, symbol M74VHC1GT66DTT1G:M74VHC1GT66DTT1G
- Q3, Q6: renamed from Q?; MPN (none) -> IRF7749L2TRPBF; category Trans -> (none); continuous drain current 36A -> (none); device class L1 Discrete Semiconductors -> (none); device class L2 Transistors -> (none); device class L3 MOSFETs -> (none); digikey description MOSFET N-CH 60V DIRECTFET L8 -> (none); digikey part number IRF7749L2TRPBFCT-ND -> (none); drain to source breakdown voltage 60V -> (none); drain to source resistance 1.1mΩ -> (none); gate to source voltage 60V -> (none); height 0.74mm -> (none); input capacitace at vds 10655pF @ 25V -> (none); lead free yes -> (none); library id f9001e01a073ea36 -> (none); manufacturer Infineon -> (none); max junction temp +175°C -> (none); mouser part number 942-IRF7749L2TRPBF -> (none); number of N channels 1 -> (none); number of channels 1 -> (none); package DirectFET -> (none); power dissipation 3.8W -> (none); rohs yes -> (none); technology MOSFET -> (none); temperature range high +175°C -> (none); temperature range low -55°C -> (none); threshold vgs 4V -> (none); turn off delay time 72ns -> (none); turn on delay time 29ns -> (none)
Connections:
- net SUPPLY: now reaches Q3.1 (D)
- net SUPPLY: now also Q3.4 (D), C1.1, C16.1, C17.1, C2.1, C3.1, C4.1, C5.1, C6.1, P1.1, Q1.1 (D), Q1.4 (D), Q2.1 (D), Q2.4 (D)
- net SH_C: now reaches Q3.10 (S)
- net SH_C: now also Q3.11 (S), Q3.2 (S), Q3.3 (S), Q3.5 (S), Q3.6 (S), Q3.8 (S), Q3.9 (S), Q6.1 (D), Q6.4 (D), R6.2, U3.8 (IN+)
- net at Q3.7 (G): now also R3.1
- net GND: now reaches Q6.10 (S)
- net GND: now also Q6.11 (S), Q6.2 (S), Q6.3 (S), Q6.5 (S), Q6.6 (S), Q6.8 (S), Q6.9 (S), C1.2, C10.1, C11.1, C12.1, C13.1, C14.1, C15.1, C16.2, C17.2, C18.1, C2.2, C3.2, C4.2, C5.2, C6.2, C7.2, C8.2, C9.2, P5.1, Q4.10 (S), Q4.11 (S), Q4.2 (S), Q4.3 (S), Q4.5 (S), Q4.6 (S), Q4.8 (S), Q4.9 (S), Q5.10 (S), Q5.11 (S), Q5.2 (S), Q5.3 (S), Q5.5 (S), Q5.6 (S), Q5.8 (S), Q5.9 (S), R14.1, U1.2 (GND), U1.3 (REF2), U2.2 (GND), U2.3 (REF2), U3.2 (GND), U3.3 (REF2), U4.3 (GND), U5.3 (GND), U6.3 (GND)
- net at Q6.7 (G): now also R9.1
- new net: P4.1, R6.1, U3.1 (IN-)
- new net: C15.2, U6.2 (OUT/INYA)
- new net: Q2.7 (G), R2.1
- new net: Q5.7 (G), R8.1
- new net: P3.1, R5.1, U2.1 (IN-)
- new net: C14.2, U5.2 (OUT/INYA)
- new net: Q1.7 (G), R1.1
- new net: Q4.7 (G), R7.1
- new net: P2.1, R4.1, U1.1 (IN-)
- new net: C13.2, U4.2 (OUT/INYA)
- new net +3V3: C7.1, C8.1, C9.1, R13.2, U1.6 (VS), U1.7 (REF1), U2.6 (VS), U2.7 (REF1), U3.6 (VS), U3.7 (REF1), U4.5 (VCC), U5.5 (VCC), U6.5 (VCC)
- new net CURR_A: C10.2, R10.2, U4.1 (IN/OUTXA)
- new net CURR_B: C11.2, R11.2, U5.1 (IN/OUTXA)
- new net CURR_C: C12.2, R12.2, U6.1 (IN/OUTXA)
- new net CURR_FILTER: U4.4 (ON/OFF), U5.4 (ON/OFF), U6.4 (ON/OFF)
- new net C_A: R10.1, U1.5 (OUT)
- new net C_B: R11.1, U2.5 (OUT)
- new net C_C: R12.1, U3.5 (OUT)
- new net GH_A: R1.2
- new net GH_B: R2.2
- new net GH_C: R3.2
- new net GL_A: R7.2
- new net GL_B: R8.2
- new net GL_C: R9.2
- new net SH_A: Q1.10 (S), Q1.11 (S), Q1.2 (S), Q1.3 (S), Q1.5 (S), Q1.6 (S), Q1.8 (S), Q1.9 (S), Q4.1 (D), Q4.4 (D), R4.2, U1.8 (IN+)
- new net SH_B: Q2.10 (S), Q2.11 (S), Q2.2 (S), Q2.3 (S), Q2.5 (S), Q2.6 (S), Q2.8 (S), Q2.9 (S), Q5.1 (D), Q5.4 (D), R5.2, U2.8 (IN+)
- new net TEMP: C18.2, R13.1, R14.2
Other:
- moved on the sheet: Q3, Q6

Commit message: 210104
Parts:
- P2, P3, P4: footprint (none) -> PADS:HighCurrent_WithHoles_250mils
Changed lines of the file:
@@
 F 0 "P4" H 7692 1885 50  0000 C CNN
 F 1 "PH_C" H 7692 1976 50  0000 C CNN
-F 2 "" H 7750 2100 50  0001 C CNN
+F 2 "PADS:HighCurrent_WithHoles_250mils" H 7750 2100 50  0001 C CNN
 F 3 "" H 7750 2100 50  0001 C CNN
 	1    7750 2100
@@
 F 0 "P3" H 4142 1885 50  0000 C CNN
 F 1 "PH_B" H 4142 1976 50  0000 C CNN
-F 2 "" H 4200 2100 50  0001 C CNN
+F 2 "PADS:HighCurrent_WithHoles_250mils" H 4200 2100 50  0001 C CNN
 F 3 "" H 4200 2100 50  0001 C CNN
 	1    4200 2100
@@
 F 0 "P2" H 592 1885 50  0000 C CNN
 F 1 "PH_A" H 592 1976 50  0000 C CNN
-F 2 "" H 650 2100 50  0001 C CNN
+F 2 "PADS:HighCurrent_WithHoles_250mils" H 650 2100 50  0001 C CNN
 F 3 "" H 650 2100 50  0001 C CNN
 	1    650  2100
