File: design/rotomdriver.sch (KiCad schematic (older format))
At the start: 0 parts

Commit message: power board design 1
Changed lines of the file:
@@
 $Descr A4 11693 8268
 encoding utf-8
-Sheet 1 2
+Sheet 1 3
 Title ""
 Date ""
@@
 $EndDescr
 $Sheet
-S 9600 2100 800  2250
+S 10000 1000 650  2600
 U 5FD2FB17
 F0 "power" 50
 F1 "power.sch" 50
+F2 "SUPPLY" I L 10000 1100 50
+F3 "GH_A" I L 10000 1400 50
+F4 "SH_A" I L 10000 1500 50
+F5 "GL_A" I L 10000 1600 50
+F6 "SL_A" I L 10000 1700 50
+F7 "GH_B" I L 10000 1900 50
+F8 "SH_B" I L 10000 2000 50
+F9 "GL_B" I L 10000 2100 50
+F10 "SL_B" I L 10000 2200 50
+F11 "GH_C" I L 10000 2400 50
+F12 "SH_C" I L 10000 2500 50
+F13 "GL_C" I L 10000 2600 50
+F14 "SL_C" I L 10000 2700 50
+F15 "CURR_FILTER" I L 10000 3100 50
+F16 "CURR_A" I L 10000 3200 50
+F17 "CURR_B" I L 10000 3300 50
+F18 "CURR_C" I L 10000 3400 50
+F19 "TEMP" I L 10000 3500 50
+$EndSheet
+$Sheet
+S 8500 1000 1000 1900
+U 5FE9ECD0
+F0 "drv8301" 50
+F1 "drv8301.sch" 50
 $EndSheet
 $EndSCHEMATC

Commit message: 210104
Parts:
- added J1: Conn_01x30_Male, Connector_PinHeader_2.54mm:PinHeader_2x15_P2.54mm_Vertical, symbol Connector:Conn_01x30_Male
Connections:
- net power/CURR_A: now also J1.22 (Pin_22)
- net power/CURR_B: now also J1.23 (Pin_23)
- net power/CURR_C: now also J1.24 (Pin_24)
- net power/CURR_FILTER: now also J1.21 (Pin_21)
- net power/TEMP: now also J1.25 (Pin_25)
- new net +3V3: J1.28 (Pin_28)
- new net +5V: J1.27 (Pin_27)
- new net EN_BUCK: J1.7 (Pin_7)
- new net GND: J1.14 (Pin_14), J1.20 (Pin_20), J1.26 (Pin_26), J1.29 (Pin_29), J1.30 (Pin_30)
- new net drv8301/CS: J1.13 (Pin_13)
- new net drv8301/EN_GATE: J1.9 (Pin_9)
- new net drv8301/FAULT: J1.8 (Pin_8)
- new net drv8301/INH_A: J1.1 (Pin_1)
- new net drv8301/INH_B: J1.2 (Pin_2)
- new net drv8301/INH_C: J1.3 (Pin_3)
- new net drv8301/INL_A: J1.4 (Pin_4)
- new net drv8301/INL_B: J1.5 (Pin_5)
- new net drv8301/INL_C: J1.6 (Pin_6)
- new net drv8301/SCLK: J1.12 (Pin_12)
- new net drv8301/SDI: J1.11 (Pin_11)
- new net drv8301/SDO: J1.10 (Pin_10)
- new net drv8301/SENS_A: J1.15 (Pin_15)
- new net drv8301/SENS_B: J1.16 (Pin_16)
- new net drv8301/SENS_C: J1.17 (Pin_17)
- new net drv8301/SENS_FILTERED: J1.19 (Pin_19)
- new net drv8301/SENS_SUPPLY: J1.18 (Pin_18)
Changed lines of the file:
@@
 $EndSheet
 $Sheet
-S 8500 1000 1000 1900
+S 8500 1000 1000 1950
 U 5FE9ECD0
 F0 "drv8301" 50
 F1 "drv8301.sch" 50
+F2 "SUPPLY" I R 9500 1100 50
+F3 "EN_BUCK" I R 9500 1250 50
+F4 "GH_A" I R 9500 1400 50
+F5 "SH_A" I R 9500 1500 50
+F6 "GL_A" I R 9500 1600 50
+F7 "SL_A" I R 9500 1700 50
+F8 "GH_B" I R 9500 1900 50
+F9 "SH_B" I R 9500 2000 50
+F10 "GL_B" I R 9500 2100 50
+F11 "SL_B" I R 9500 2200 50
+F12 "GH_C" I R 9500 2400 50
+F13 "SH_C" I R 9500 2500 50
+F14 "GL_C" I R 9500 2600 50
+F15 "SL_C" I R 9500 2700 50
+F16 "INH_A" I L 8500 1100 50
+F17 "INH_B" I L 8500 1200 50
+F18 "INH_C" I L 8500 1300 50
+F19 "INL_A" I L 8500 1400 50
+F20 "INL_B" I L 8500 1500 50
+F21 "INL_C" I L 8500 1600 50
+F22 "FAULT" I L 8500 1750 50
+F23 "EN_GATE" I L 8500 1850 50
+F24 "SDO" I L 8500 2000 50
+F25 "SDI" I L 8500 2100 50
+F26 "SCLK" I L 8500 2200 50
+F27 "CS" I L 8500 2300 50
+F28 "SENS_A" I L 8500 2450 50
+F29 "SENS_B" I L 8500 2550 50
+F30 "SENS_C" I L 8500 2650 50
+F31 "SENS_SUPPLY" I L 8500 2750 50
+F32 "SENS_FILTERED" I L 8500 2850 50
 $EndSheet
+Wire Wire Line
+	9500 1100 10000 1100
+Text Label 9500 1250 0    50   ~ 0
+EN_BUCK
+Wire Wire Line
+	9500 1400 10000 1400
+Wire Wire Line
+	9500 1600 10000 1600
+Wire Wire Line
+	10000 1700 9500 1700
+Wire Wire Line
+	9500 1900 10000 1900
+Wire Wire Line
+	10000 2000 9500 2000
+Wire Wire Line
+	9500 2100 10000 2100
+Wire Wire Line
+	10000 2200 9500 2200
+Wire Wire Line
+	9500 2400 10000 2400
+Wire Wire Line
+	10000 2500 9500 2500
+Wire Wire Line
+	9500 2600 10000 2600
+Wire Wire Line
+	10000 2700 9500 2700
+Connection ~ 9750 1500
+Text Label 9750 1350 0    50   ~ 0
+SH_A
+Wire Wire Line
+	9750 1500 9750 1350
+Wire Wire Line
+	9750 1500 9500 1500
+Wire Wire Line
+	9750 1500 10000 1500
+$Comp
+L power:+5V #PWR056
+U 1 1 5FF07B73
+P 8500 3700
+F 0 "#PWR056" H 8500 3550 50  0001 C CNN
+F 1 "+5V" V 8515 3828 50  0000 L CNN
+F 2 "" H 8500 3700 50  0001 C CNN
+F 3 "" H 8500 3700 50  0001 C CNN
+	1    8500 3700
+	0    1    1    0
+$EndComp
+$Comp
+L power:+3.3V #PWR057
+U 1 1 5FF07D9F
+P 8500 3800
+F 0 "#PWR057" H 8500 3650 50  0001 C CNN
+F 1 "+3.3V" V 8515 3928 50  0000 L CNN
+F 2 "" H 8500 3800 50  0001 C CNN
+F 3 "" H 8500 3800 50  0001 C CNN
+	1    8500 3800
+	0    1    1    0
+$EndComp
+$Comp
+L power:GND #PWR058
+U 1 1 5FF212C4
+P 8500 4000
+F 0 "#PWR058" H 8500 3750 50  0001 C CNN
+F 1 "GND" H 8505 3827 50  0000 C CNN
+F 2 "" H 8500 4000 50  0001 C CNN
+F 3 "" H 8500 4000 50  0001 C CNN
+	1    8500 4000
+	1    0    0    -1
+$EndComp
+Wire Wire Line
+	8500 3900 8500 4000
+Connection ~ 8500 4000
+$Comp
+L Connector:Conn_01x30_Male J1
+U 1 1 5FF9EDA6
+P 7800 2500
+F 0 "J1" H 7908 4081 50  0000 C CNN
+F 1 "Conn_01x30_Male" H 7908 3990 50  0000 C CNN
+F 2 "Connector_PinHeader_2.54mm:PinHeader_2x15_P2.54mm_Vertical" H 7800 2500 50  0001 C CNN
+F 3 "~" H 7800 2500 50  0001 C CNN
+	1    7800 2500
+	1    0    0    -1
+$EndComp
+Wire Wire Line
+	8000 1100 8500 1100
+Wire Wire Line
+	8500 1200 8000 1200
+Wire Wire Line
+	8000 1300 8500 1300
+Wire Wire Line
+	8500 1400 8000 1400
+Wire Wire Line
+	8000 1500 8500 1500
+Wire Wire Line
+	8500 1600 8000 1600
+Wire Wire Line
+	8300 1850 8300 1900
+Wire Wire Line
+	8300 1900 8000 1900
+Wire Wire Line
+	8200 1800 8200 1750
+Wire Wire Line
+	8200 1750 8500 1750
+Wire Wire Line
+	8500 1850 8300 1850
+Wire Wire Line
+	8200 1800 8000 1800
+Wire Wire Line
+	8000 2000 8500 2000
+Wire Wire Line
+	8500 2100 8000 2100
+Wire Wire Line
+	8000 2200 8500 2200
+Wire Wire Line
+	8500 2300 8000 2300
+Wire Wire Line
+	10000 3100 8000 3100
+Wire Wire Line
+	8000 3200 10000 3200
+Wire Wire Line
+	10000 3300 8000 3300
+Wire Wire Line
+	8000 3400 10000 3400
+Wire Wire Line
+	10000 3500 8000 3500
+Wire Wire Line
+	8000 2900 8400 2900
+Wire Wire Line
+	8400 2900 8400 2850
+Wire Wire Line
+	8400 2850 8500 2850
+Wire Wire Line
+	8350 2750 8350 2800
+Wire Wire Line
+	8350 2800 8000 2800
+Wire Wire Line
+	8500 2750 8350 2750
+Wire Wire Line
+	8000 2500 8100 2500
+Wire Wire Line
+	8100 2500 8100 2450
+Wire Wire Line
+	8100 2450 8500 2450
+Wire Wire Line
+	8500 2550 8200 2550
+Wire Wire Line
+	8200 2550 8200 2600
+Wire Wire Line
+	8000 2600 8200 2600
+Wire Wire Line
+	8300 2700 8300 2650
+Wire Wire Line
+	8300 2650 8500 2650
+Wire Wire Line
+	8000 2700 8300 2700
+Wire Wire Line
+	8000 3700 8500 3700
+Wire Wire Line
+	8000 3800 8500 3800
+Wire Wire Line
+	8000 3900 8500 3900
+Wire Wire Line
+	8000 4000 8500 4000
+Text Label 8000 1700 0    50   ~ 0
+EN_BUCK
+$Comp
+L power:GND #PWR?
+U 1 1 6011161C
+P 8000 2400
+F 0 "#PWR?" H 8000 2150 50  0001 C CNN
+F 1 "GND" V 8005 2227 50  0000 C CNN
+F 2 "" H 8000 2400 50  0001 C CNN
+F 3 "" H 8000 2400 50  0001 C CNN
+	1    8000 2400
+	0    -1   -1   0
+$EndComp
+$Comp
+L power:GND #PWR?
+U 1 1 6011232F
+P 8000 3000
+F 0 "#PWR?" H 8000 2750 50  0001 C CNN
+F 1 "GND" V 8005 2827 50  0000 C CNN
+F 2 "" H 8000 3000 50  0001 C CNN
+F 3 "" H 8000 3000 50  0001 C CNN
+	1    8000 3000
+	0    -1   -1   0
+$EndComp
+$Comp
+L power:GND #PWR?
+U 1 1 6011277E
+P 8000 3600
+F 0 "#PWR?" H 8000 3350 50  0001 C CNN
+F 1 "GND" V 8005 3427 50  0000 C CNN
+F 2 "" H 8000 3600 50  0001 C CNN
+F 3 "" H 8000 3600 50  0001 C CNN
+	1    8000 3600
+	0    -1   -1   0
+$EndComp
 $EndSCHEMATC
